File: pcb2/shield/shield.sch (KiCad schematic (older format))
At the start: 29 parts, among them IC1 STM32F0xxKxTx, IC2 MCP1700, IC3 AM26C31, IC4 AM26C31, J1 MICROUSB, P1 SWD_TC, P10 BUS5, P11 BUS6, P12 BUS7, P13 BUS8, P5 SHIFT, P6 BUS1, P7 BUS2, P8 BUS3, P9 BUS4, X1 PART, X2 PART, X3 PART, X4 PART

Commit message: shield PCB ERC
Connections:
- no-connect marks 5 -> 22
Changed lines of the file:
@@
 $EndComp
 $Comp
-L GND #PWR30
+L GND #PWR01
 U 1 1 56F85F2A
 P 8850 1650
-F 0 "#PWR30" H 8850 1400 50  0001 C CNN
+F 0 "#PWR01" H 8850 1400 50  0001 C CNN
 F 1 "GND" H 8850 1500 50  0000 C CNN
 F 2 "" H 8850 1650 50  0000 C CNN
@@
 $EndComp
 $Comp
-L +5V #PWR25
+L +5V #PWR02
 U 1 1 56F86D5E
 P 8200 2300
-F 0 "#PWR25" H 8200 2150 50  0001 C CNN
+F 0 "#PWR02" H 8200 2150 50  0001 C CNN
 F 1 "+5V" H 8200 2440 50  0000 C CNN
 F 2 "" H 8200 2300 50  0000 C CNN
@@
 $EndComp
 $Comp
-L GND #PWR26
+L GND #PWR03
 U 1 1 56F86DAA
 P 8250 2500
-F 0 "#PWR26" H 8250 2250 50  0001 C CNN
+F 0 "#PWR03" H 8250 2250 50  0001 C CNN
 F 1 "GND" H 8250 2350 50  0000 C CNN
 F 2 "" H 8250 2500 50  0000 C CNN
@@
 $EndComp
 $Comp
-L +5V #PWR24
+L +5V #PWR04
 U 1 1 56F86E73
 P 7950 3900
-F 0 "#PWR24" H 7950 3750 50  0001 C CNN
+F 0 "#PWR04" H 7950 3750 50  0001 C CNN
 F 1 "+5V" H 7950 4040 50  0000 C CNN
 F 2 "" H 7950 3900 50  0000 C CNN
@@
 $EndComp
 $Comp
-L GND #PWR27
+L GND #PWR05
 U 1 1 56F86EC2
 P 8250 4100
-F 0 "#PWR27" H 8250 3850 50  0001 C CNN
+F 0 "#PWR05" H 8250 3850 50  0001 C CNN
 F 1 "GND" H 8250 3950 50  0000 C CNN
 F 2 "" H 8250 4100 50  0000 C CNN
@@
 NoConn ~ 8350 2700
 $Comp
-L GND #PWR28
+L GND #PWR06
 U 1 1 56F87C8E
 P 8350 2800
-F 0 "#PWR28" H 8350 2550 50  0001 C CNN
+F 0 "#PWR06" H 8350 2550 50  0001 C CNN
 F 1 "GND" H 8350 2650 50  0001 C CNN
 F 2 "" H 8350 2800 50  0000 C CNN
@@
 $EndComp
 $Comp
-L GND #PWR29
+L GND #PWR07
 U 1 1 56F87D9A
 P 8350 4400
-F 0 "#PWR29" H 8350 4150 50  0001 C CNN
+F 0 "#PWR07" H 8350 4150 50  0001 C CNN
 F 1 "GND" H 8350 4250 50  0001 C CNN
 F 2 "" H 8350 4400 50  0000 C CNN
@@
 $EndComp
 $Comp
-L +5V #PWR15
+L +5V #PWR08
 U 1 1 5794B897
-P 4550 1300
-F 0 "#PWR15" H 4550 1150 50  0001 C CNN
-F 1 "+5V" H 4565 1473 50  0000 C CNN
-F 2 "" H 4550 1300 50  0000 C CNN
-F 3 "" H 4550 1300 50  0000 C CNN
-	1    4550 1300
-	1    0    0    -1
-$EndComp
-$Comp
-L GND #PWR16
+P 4800 1300
+F 0 "#PWR08" H 4800 1150 50  0001 C CNN
+F 1 "+5V" H 4815 1473 50  0000 C CNN
+F 2 "" H 4800 1300 50  0000 C CNN
+F 3 "" H 4800 1300 50  0000 C CNN
+	1    4800 1300
+	1    0    0    -1
+$EndComp
+$Comp
+L GND #PWR09
 U 1 1 5794B8F4
-P 4600 1950
-F 0 "#PWR16" H 4600 1700 50  0001 C CNN
-F 1 "GND" H 4605 1777 50  0000 C CNN
-F 2 "" H 4600 1950 50  0000 C CNN
-F 3 "" H 4600 1950 50  0000 C CNN
-	1    4600 1950
-	1    0    0    -1
-$EndComp
-$Comp
-L +3V3 #PWR12
+P 4800 1950
+F 0 "#PWR09" H 4800 1700 50  0001 C CNN
+F 1 "GND" H 4805 1777 50  0000 C CNN
+F 2 "" H 4800 1950 50  0000 C CNN
+F 3 "" H 4800 1950 50  0000 C CNN
+	1    4800 1950
+	1    0    0    -1
+$EndComp
+$Comp
+L +3V3 #PWR010
 U 1 1 5794BB55
 P 2500 3200
-F 0 "#PWR12" H 2500 3050 50  0001 C CNN
+F 0 "#PWR010" H 2500 3050 50  0001 C CNN
 F 1 "+3V3" H 2515 3373 50  0000 C CNN
 F 2 "" H 2500 3200 50  0000 C CNN
@@
 $EndComp
 $Comp
-L GND #PWR9
+L GND #PWR011
 U 1 1 5794BBFE
 P 2400 3550
-F 0 "#PWR9" H 2400 3300 50  0001 C CNN
+F 0 "#PWR011" H 2400 3300 50  0001 C CNN
 F 1 "GND" H 2405 3377 50  0000 C CNN
 F 2 "" H 2400 3550 50  0000 C CNN
@@
 $EndComp
 $Comp
-L GND #PWR5
+L GND #PWR012
 U 1 1 5794BE19
 P 1850 4150
-F 0 "#PWR5" H 1850 3900 50  0001 C CNN
+F 0 "#PWR012" H 1850 3900 50  0001 C CNN
 F 1 "GND" H 1855 3977 50  0000 C CNN
 F 2 "" H 1850 4150 50  0000 C CNN
@@
 nRST
 $Comp
-L GND #PWR8
+L GND #PWR013
 U 1 1 5794BF98
 P 2150 3950
-F 0 "#PWR8" H 2150 3700 50  0001 C CNN
+F 0 "#PWR013" H 2150 3700 50  0001 C CNN
 F 1 "GND" H 2155 3777 50  0000 C CNN
 F 2 "" H 2150 3950 50  0000 C CNN
@@
 $EndComp
 $Comp
-L +3V3 #PWR1
+L +3V3 #PWR014
 U 1 1 5794C2DC
 P 1350 900
-F 0 "#PWR1" H 1350 750 50  0001 C CNN
+F 0 "#PWR014" H 1350 750 50  0001 C CNN
 F 1 "+3V3" H 1365 1073 50  0000 C CNN
 F 2 "" H 1350 900 50  0000 C CNN
@@
 $EndComp
 $Comp
-L +3V3 #PWR3
+L +3V3 #PWR015
 U 1 1 5794C329
 P 1750 900
-F 0 "#PWR3" H 1750 750 50  0001 C CNN
+F 0 "#PWR015" H 1750 750 50  0001 C CNN
 F 1 "+3V3" H 1765 1073 50  0000 C CNN
 F 2 "" H 1750 900 50  0000 C CNN
@@
 $EndComp
 $Comp
-L +3V3 #PWR6
+L +3V3 #PWR016
 U 1 1 5794C376
 P 2100 900
-F 0 "#PWR6" H 2100 750 50  0001 C CNN
+F 0 "#PWR016" H 2100 750 50  0001 C CNN
 F 1 "+3V3" H 2115 1073 50  0000 C CNN
 F 2 "" H 2100 900 50  0000 C CNN
@@
 $EndComp
 $Comp
-L GND #PWR2
+L GND #PWR017
 U 1 1 5794C3C3
 P 1350 1200
-F 0 "#PWR2" H 1350 950 50  0001 C CNN
+F 0 "#PWR017" H 1350 950 50  0001 C CNN
 F 1 "GND" H 1355 1027 50  0000 C CNN
 F 2 "" H 1350 1200 50  0000 C CNN
@@
 $EndComp
 $Comp
-L GND #PWR4
+L GND #PWR018
 U 1 1 5794C410
 P 1750 1200
-F 0 "#PWR4" H 1750 950 50  0001 C CNN
+F 0 "#PWR018" H 1750 950 50  0001 C CNN
 F 1 "GND" H 1755 1027 50  0000 C CNN
 F 2 "" H 1750 1200 50  0000 C CNN
@@
 $EndComp
 $Comp
-L GND #PWR7
+L GND #PWR019
 U 1 1 5794C45D
 P 2100 1200
-F 0 "#PWR7" H 2100 950 50  0001 C CNN
+F 0 "#PWR019" H 2100 950 50  0001 C CNN
 F 1 "GND" H 2105 1027 50  0000 C CNN
 F 2 "" H 2100 1200 50  0000 C CNN
@@
 $EndComp
 $Comp
-L +3V3 #PWR10
+L +3V3 #PWR020
 U 1 1 5794C73B
 P 2500 900
-F 0 "#PWR10" H 2500 750 50  0001 C CNN
+F 0 "#PWR020" H 2500 750 50  0001 C CNN
 F 1 "+3V3" H 2515 1073 50  0000 C CNN
 F 2 "" H 2500 900 50  0000 C CNN
@@
 $EndComp
 $Comp
-L +3V3 #PWR13
+L +3V3 #PWR021
 U 1 1 5794C78E
 P 2800 900
-F 0 "#PWR13" H 2800 750 50  0001 C CNN
+F 0 "#PWR021" H 2800 750 50  0001 C CNN
 F 1 "+3V3" H 2815 1073 50  0000 C CNN
 F 2 "" H 2800 900 50  0000 C CNN
@@
 $EndComp
 $Comp
-L GND #PWR11
+L GND #PWR022
 U 1 1 5794C7E1
 P 2500 1200
-F 0 "#PWR11" H 2500 950 50  0001 C CNN
+F 0 "#PWR022" H 2500 950 50  0001 C CNN
 F 1 "GND" H 2505 1027 50  0000 C CNN
 F 2 "" H 2500 1200 50  0000 C CNN
@@
 $EndComp
 $Comp
-L GND #PWR14
+L GND #PWR023
 U 1 1 5794C834
 P 2800 1200
-F 0 "#PWR14" H 2800 950 50  0001 C CNN
+F 0 "#PWR023" H 2800 950 50  0001 C CNN
 F 1 "GND" H 2805 1027 50  0000 C CNN
 F 2 "" H 2800 1200 50  0000 C CNN
@@
 $EndComp
 $Comp
-L GND #PWR21
+L GND #PWR024
 U 1 1 5794D178
 P 6000 1450
-F 0 "#PWR21" H 6000 1200 50  0001 C CNN
+F 0 "#PWR024" H 6000 1200 50  0001 C CNN
 F 1 "GND" H 6005 1277 50  0000 C CNN
 F 2 "" H 6000 1450 50  0000 C CNN
@@
 	8150 3900 7950 3900
 Wire Wire Line
-	4550 1300 4550 1350
-Wire Wire Line
-	4550 1350 4450 1350
-Wire Wire Line
-	4450 1750 4600 1750
-Wire Wire Line
-	4600 1750 4600 1950
+	4800 1350 4800 1300
+Wire Wire Line
+	4450 1350 4800 1350
+Wire Wire Line
+	4450 1750 4800 1750
+Wire Wire Line
+	4800 1750 4800 1950
 Wire Wire Line
 	2500 3200 2500 3450
@@
 	2150 3950 2600 3950
 $Comp
-L +5V #PWR19
+L +5V #PWR025
 U 1 1 5794D32F
 P 5600 1350
-F 0 "#PWR19" H 5600 1200 50  0001 C CNN
+F 0 "#PWR025" H 5600 1200 50  0001 C CNN
 F 1 "+5V" H 5615 1523 50  0000 C CNN
 F 2 "" H 5600 1350 50  0000 C CNN
@@
 Connection ~ 5600 1350
 $Comp
-L GND #PWR20
+L GND #PWR026
 U 1 1 5794D41F
 P 5600 1650
-F 0 "#PWR20" H 5600 1400 50  0001 C CNN
+F 0 "#PWR026" H 5600 1400 50  0001 C CNN
 F 1 "GND" H 5605 1477 50  0000 C CNN
 F 2 "" H 5600 1650 50  0000 C CNN
@@
 $EndComp
 $Comp
-L +3V3 #PWR22
+L +3V3 #PWR027
 U 1 1 5794D4F1
 P 6900 1350
-F 0 "#PWR22" H 6900 1200 50  0001 C CNN
+F 0 "#PWR027" H 6900 1200 50  0001 C CNN
 F 1 "+3V3" H 6915 1523 50  0000 C CNN
 F 2 "" H 6900 1350 50  0000 C CNN
@@
 Connection ~ 6900 1350
 $Comp
-L GND #PWR23
+L GND #PWR028
 U 1 1 5794D58E
 P 6900 1650
-F 0 "#PWR23" H 6900 1400 50  0001 C CNN
+F 0 "#PWR028" H 6900 1400 50  0001 C CNN
 F 1 "GND" H 6905 1477 50  0000 C CNN
 F 2 "" H 6900 1650 50  0000 C CNN
@@
 $EndComp
 $Comp
-L +3V3 #PWR17
+L +3V3 #PWR029
 U 1 1 5794F9F0
 P 5450 5200
-F 0 "#PWR17" H 5450 5050 50  0001 C CNN
+F 0 "#PWR029" H 5450 5050 50  0001 C CNN
 F 1 "+3V3" H 5465 5373 50  0000 C CNN
 F 2 "" H 5450 5200 50  0000 C CNN
@@
 $EndComp
 $Comp
-L GND #PWR18
+L GND #PWR030
 U 1 1 5794FA4F
 P 5450 5400
-F 0 "#PWR18" H 5450 5150 50  0001 C CNN
+F 0 "#PWR030" H 5450 5150 50  0001 C CNN
 F 1 "GND" H 5455 5227 50  0000 C CNN
 F 2 "" H 5450 5400 50  0000 C CNN
@@
 Text Notes 900  6400 0    60   ~ 0
 Mounting\nHoles
+NoConn ~ 2600 4150
+NoConn ~ 2600 4250
+NoConn ~ 2600 4450
+NoConn ~ 2600 4550
+NoConn ~ 2600 4750
+NoConn ~ 2600 4850
+NoConn ~ 2600 4950
+NoConn ~ 2600 5050
+NoConn ~ 2600 5150
+NoConn ~ 3400 3250
+NoConn ~ 3400 3350
+NoConn ~ 3400 3550
+NoConn ~ 3400 3650
+NoConn ~ 3400 4050
+NoConn ~ 3400 4150
+NoConn ~ 3400 4250
+NoConn ~ 3400 4750
+$Comp
+L PWR_FLAG #FLG031
+U 1 1 57957B1B
+P 4600 1250
+F 0 "#FLG031" H 4600 1345 50  0001 C CNN
+F 1 "PWR_FLAG" H 4600 1474 50  0000 C CNN
+F 2 "" H 4600 1250 50  0000 C CNN
+F 3 "" H 4600 1250 50  0000 C CNN
+	1    4600 1250
+	1    0    0    -1
+$EndComp
+Wire Wire Line
+	4600 1250 4600 1350
+Connection ~ 4600 1350
+$Comp
+L PWR_FLAG #FLG032
+U 1 1 57957C2A
+P 4600 2000
+F 0 "#FLG032" H 4600 2095 50  0001 C CNN
+F 1 "PWR_FLAG" H 4600 2223 50  0000 C CNN
+F 2 "" H 4600 2000 50  0000 C CNN
+F 3 "" H 4600 2000 50  0000 C CNN
+	1    4600 2000
+	-1   0    0    1
+$EndComp
+Wire Wire Line
+	4600 2000 4600 1750
+Connection ~ 4600 1750
 $EndSCHEMATC

Commit message: Added parts, BOM and stickerBOM
Parts:
- C1, C2: Farnell 2496833 -> 2524817
- C10, C7, C9: Farnell (none) -> 2524858
- C3, C6, C8: Farnell (none) -> 2524817
- C4: Farnell (none) -> 2494230
- C5: value C -> 100n; Farnell (none) -> 2524817
Changed lines of the file:
@@
 F 2 "agg:0603" H 8200 2400 50  0001 C CNN
 F 3 "" H 8200 2400 50  0000 C CNN
-F 4 "2496833" H 8200 2400 60  0001 C CNN "Farnell"
+F 4 "2524817" H 8200 2400 60  0001 C CNN "Farnell"
 	1    8200 2400
 	1    0    0    -1
@@
 F 2 "agg:0603" H 7950 4000 50  0001 C CNN
 F 3 "" H 7950 4000 50  0000 C CNN
-F 4 "2496833" H 7950 4000 60  0001 C CNN "Farnell"
+F 4 "2524817" H 7950 4000 60  0001 C CNN "Farnell"
 	1    7950 4000
 	1    0    0    -1
@@
 P 1850 4000
 F 0 "C5" H 1965 4046 50  0000 L CNN
-F 1 "C" H 1965 3955 50  0000 L CNN
+F 1 "100n" H 1965 3955 50  0000 L CNN
 F 2 "agg:0603" H 1888 3850 50  0001 C CNN
 F 3 "" H 1850 4000 50  0000 C CNN
+F 4 "2524817" H 1850 4000 60  0001 C CNN "Farnell"
 	1    1850 4000
 	1    0    0    -1
@@
 F 2 "agg:0603" H 1465 959 50  0001 L CNN
 F 3 "" H 1350 1050 50  0000 C CNN
+F 4 "2524817" H 1350 1050 60  0001 C CNN "Farnell"
 	1    1350 1050
 	1    0    0    -1
@@
 F 2 "agg:0603" H 1788 900 50  0001 C CNN
 F 3 "" H 1750 1050 50  0000 C CNN
+F 4 "2494230" H 1750 1050 60  0001 C CNN "Farnell"
 	1    1750 1050
 	1    0    0    -1
@@
 F 2 "agg:0603" H 2138 900 50  0001 C CNN
 F 3 "" H 2100 1050 50  0000 C CNN
+F 4 "2524817" H 2100 1050 60  0001 C CNN "Farnell"
 	1    2100 1050
 	1    0    0    -1
@@
 F 2 "agg:0603" H 2538 900 50  0001 C CNN
 F 3 "" H 2500 1050 50  0000 C CNN
+F 4 "2524858" H 2500 1050 60  0001 C CNN "Farnell"
 	1    2500 1050
 	1    0    0    -1
@@
 F 2 "agg:0603" H 2838 900 50  0001 C CNN
 F 3 "" H 2800 1050 50  0000 C CNN
+F 4 "2524817" H 2800 1050 60  0001 C CNN "Farnell"
 	1    2800 1050
 	1    0    0    -1
@@
 F 2 "agg:0603" H 5638 1350 50  0001 C CNN
 F 3 "" H 5600 1500 50  0000 C CNN
+F 4 "2524858" H 5600 1500 60  0001 C CNN "Farnell"
 	1    5600 1500
 	1    0    0    -1
@@
 F 2 "agg:0603" H 6938 1350 50  0001 C CNN
 F 3 "" H 6900 1500 50  0000 C CNN
+F 4 "2524858" H 6900 1500 60  0001 C CNN "Farnell"
 	1    6900 1500
 	1    0    0    -1
